File: PCB/Eagle/sFPI-Driver/sFPI-Driver.sch (EAGLE design)
At the start: 3 parts, among them IC1 ATMEGA168-PU, IC2 LM741P

Commit message: Eagle Layout UPDATE - LTSPICE UPDATE
Parts:
- removed IC2: LM741P, linear:LM741P
- added R1, R3, R5: (no value), resistor:R-TRIMM74X
- added R12, R14, R2, R4, R6, R9: (no value), rcl:R-US_M1206
- added U1: LT1006CN8PBF, LTC:LT1006CN8PBF
Changed lines of the file:
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@@
 <layer number="97" name="Info" color="7" fill="1" visible="yes" active="yes"/>
 <layer number="98" name="Guide" color="6" fill="1" visible="yes" active="yes"/>
+<layer number="99" name="SpiceOrder" color="5" fill="1" visible="yes" active="yes"/>
 </layers>
 <schematic xreflabel="%F%N/%S.%C%R" xrefpart="/%S.%C%R">
@@
 <part name="IC1" library="Arduino-AVR" deviceset="ATMEGA168-PU" device=""/>
 <part name="QF1" library="crystal" deviceset="16M20AUM1" device=""/>
-<part name="IC2" library="linear" deviceset="*741" device="P" technology="LM"/>
+<part name="U1" library="LTC" deviceset="LT1006CN8PBF" device=""/>
+<part name="R4" library="rcl" deviceset="R-US_" device="M1206"/>
+<part name="R2" library="rcl" deviceset="R-US_" device="M1206"/>
+<part name="R6" library="rcl" deviceset="R-US_" device="M1206"/>
+<part name="R9" library="rcl" deviceset="R-US_" device="M1206"/>
+<part name="R12" library="rcl" deviceset="R-US_" device="M1206"/>
+<part name="R14" library="rcl" deviceset="R-US_" device="M1206"/>
+<part name="R1" library="resistor" deviceset="R-TRIMM" device="74X"/>
+<part name="R3" library="resistor" deviceset="R-TRIMM" device="74X"/>
+<part name="R5" library="resistor" deviceset="R-TRIMM" device="74X"/>
 </parts>
 <sheets>
@@
 <instance part="IC1" gate="1" x="22.86" y="60.96"/>
 <instance part="QF1" gate="G$1" x="-17.78" y="71.12" rot="R270"/>
-<instance part="IC2" gate="A" x="114.3" y="71.12"/>
+<instance part="U1" gate="A" x="111.76" y="78.74"/>
+<instance part="R4" gate="G$1" x="152.4" y="93.98"/>
+<instance part="R2" gate="G$1" x="86.36" y="93.98" rot="R90"/>
+<instance part="R6" gate="G$1" x="154.94" y="111.76"/>
+<instance part="R9" gate="G$1" x="147.32" y="43.18" rot="R180"/>
+<instance part="R12" gate="G$1" x="147.32" y="58.42" rot="R180"/>
+<instance part="R14" gate="G$1" x="144.78" y="71.12" rot="R180"/>
+<instance part="R1" gate="G$1" x="93.98" y="114.3" rot="R270"/>
+<instance part="R3" gate="G$1" x="124.46" y="109.22"/>
+<instance part="R5" gate="G$1" x="137.16" y="116.84"/>
 </instances>
 <busses>
