File: PCB/Eagle/sFPI-Driver/sFPI-Driver.sch (EAGLE design)
At the start: 19 parts, among them IC1 ATMEGA168-PU

Commit message: sFPI - Rev 1
Parts:
- removed R13: 10k, resistor:R-TRIMM74X
- added C3, C4: 1u, rcl:C-US050-030X075
- added OPAMP5, OPAMP6: LT1006CN8PBF, LTC:LT1006CN8PBF
- added R11, R4: (no value), rcl:POTENTIOMETER_PT-10
- added R5, R6, R9: 10k, rcl:R-US_M1206
- added VR2: LT3080-SOT223, sFPI:LT3080-SOT223
- R1: value 100k -> (none); device resistor:R-TRIMM74X -> rcl:POTENTIOMETER_PT-10
- R7: value 10k -> (none); device resistor:R-TRIMM74X -> rcl:POTENTIOMETER_PT-10
Connections:
- removed net N$13: R7.S
- removed net N$3: R1.S
- new net N$19: OPAMP6.-IN, R5.1, R6.1, R9.2
- new net N$20: C4.1, OPAMP5.+IN, VR2.VO
- new net N$23: R4.2, VR2.SET
- new net N$24: OPAMP4.-IN, OPAMP4.OUT, R5.2
- new net N$25: OPAMP6.OUT, R9.1
- net GND: now also OPAMP6.+IN
- net N$10: now also R11.3; no longer R1.A
- net N$12: now also R1.2, R7.2; no longer R7.E
- net N$17: now also OPAMP5.-IN, OPAMP5.OUT, R6.2; no longer OPAMP4.-IN, OPAMP4.OUT
- net N$5: now also R1.3, R7.3; no longer R7.A
- net N$9: now also R11.2; no longer R1.E
- net V+: now also C3.1, OPAMP5.V+, OPAMP6.V+, VR2.VI
- net V-: now also C3.2, C4.2, OPAMP5.V-, OPAMP6.V-, R4.3

Commit message: sFPI - Rev 2
Parts:
- added C5, C6: (no value), rcl:C-US050-025X075
- added R12: 10k, rcl:R-US_M1206
- renumbered OPAMP1 to U1, OPAMP2 to U2, OPAMP3 to U3, OPAMP4 to U4, OPAMP5 to U5, OPAMP6 to U6
Connections:
- net N$25 renamed V_PZT
- new net N$3: IC1.RESET, R12.1
- net GND: now also C5.2, C6.2
- net N$1: now also C5.1
- net N$2: now also C6.1
- net N$4: now also R12.2

Commit message: sFPI - Updated Parts List - Updated LTSpice Models and Scripts
Parts:
- removed R11: (no value), rcl:POTENTIOMETER_PT-10
- removed R12, R16: 10k, rcl:R-US_M1206
- removed R15: 3.3k, rcl:R-US_M1206
- added C7, C8, C9: CAP-CER-22PF-50V-NP0-RADIAL, sFPI:CAP-CER-22PF-50V-NP0-RADIAL
- added T1, T2, T3, T4: POTMILRV8-SPR, sFPI:POTMILRV8-SPR
- C5, C6: value (none) -> CAP-CER-22PF-50V-NP0-RADIAL; device rcl:C-US050-025X075 -> sFPI:CAP-CER-22PF-50V-NP0-RADIAL
- R1, R4: value (none) -> 10k; device rcl:POTENTIOMETER_PT-10 -> rcl:R-US_M1206
- R3, R5: value 10k -> 3.3k
- R7: value (none) -> 1M; device rcl:POTENTIOMETER_PT-10 -> rcl:R-US_M1206
- R8: value 3.3k -> 1M
- R9: value 10k -> 1M
Connections:
- new net N$13: R5.2, T3.2
- net GND: now also C5.1, C6.1, C7.1, C8.1, C9.1; no longer C5.2, C6.2
- net N$1: now also C5.2; no longer C5.1
- net N$10: now also R1.2, T1.2; no longer C2.+, R11.3
- net N$12: now also R3.2, T2.2; no longer R1.2, R15.2, R7.2, R8.2
- net N$14: now also C9.2, R5.1, R6.2; no longer R15.1, R16.2
- net N$16: now also R6.1; no longer R16.1
- net N$17: now also R8.2; no longer R6.2
- net N$19: now also R7.1, R8.1; no longer R5.1, R6.1
- net N$2: now also C6.2; no longer C6.1
- net N$23: now also T4.2; no longer R4.2
- net N$24: now also R7.2; no longer R5.2
- net N$3: now also R10.1; no longer R12.1
- net N$4: now also R10.2; no longer R12.2
- net N$5: now also R2.1, T2.3, T3.3; no longer R1.3, R3.1, R7.3
- net N$6: now also C7.2, C8.2, R1.1, R2.2, R3.1, R4.2; no longer R10.2, R2.1, R3.2, R8.1
- net N$9: now also C2.+, T1.3; no longer R11.2, R2.2
- net V-: now also T4.3; no longer R4.3
Other:
- moved on the sheet: R10, R2, R3, R5, R6, R8

Commit message: Final Revision
Parts:
- R1, R2, R4, R6: device rcl:R-US_M1206 -> rcl:R-US_0207/10
Connections:
- net N$10: now also R1.1, T3.2; no longer R1.2, T1.2
- net N$13: now also T1.2; no longer T3.2
- net N$14: now also R6.1; no longer R6.2
- net N$16: now also R6.2; no longer R6.1
- net N$5: now also R2.2, R4.2, T1.3; no longer R2.1, T3.3
- net N$6: now also R1.2, R2.1, R4.1; no longer R1.1, R2.2, R4.2
- net N$9: now also T3.3; no longer T1.3
Other:
- moved on the sheet: R1, R2, R4, R6, T1, T3

Commit message: ReEdited Paper with final changes
Parts:
- C5, C6: value CAP-CER-22PF-50V-NP0-RADIAL -> (none); device sFPI:CAP-CER-22PF-50V-NP0-RADIAL -> rcl:C-US025-024X044
Changed lines of the file:
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@@
 <part name="C8" library="sFPI" deviceset="CAP-CER-22PF-50V-NP0-RADIAL" device=""/>
 <part name="C9" library="sFPI" deviceset="CAP-CER-22PF-50V-NP0-RADIAL" device=""/>
-<part name="C5" library="sFPI" deviceset="CAP-CER-22PF-50V-NP0-RADIAL" device=""/>
-<part name="C6" library="sFPI" deviceset="CAP-CER-22PF-50V-NP0-RADIAL" device=""/>
 <part name="R1" library="rcl" deviceset="R-US_" device="0207/10" value="10k"/>
 <part name="R2" library="rcl" deviceset="R-US_" device="0207/10" value="10k"/>
@@
 <part name="T2" library="sFPI" deviceset="POTMILRV8" device="-SPR"/>
 <part name="T3" library="sFPI" deviceset="POTMILRV8" device="-SPR"/>
+<part name="C5" library="rcl" deviceset="C-US" device="025-024X044"/>
+<part name="C6" library="rcl" deviceset="C-US" device="025-024X044"/>
 </parts>
 <sheets>
@@
 <instance part="C8" gate="G$1" x="213.36" y="91.44"/>
 <instance part="C9" gate="G$1" x="299.72" y="91.44"/>
-<instance part="C5" gate="G$1" x="-30.48" y="81.28" rot="R90"/>
-<instance part="C6" gate="G$1" x="-30.48" y="66.04" rot="R90"/>
 <instance part="R1" gate="G$1" x="132.08" y="76.2"/>
 <instance part="R2" gate="G$1" x="157.48" y="99.06"/>
@@
 <instance part="T2" gate="G$1" x="198.12" y="83.82"/>
 <instance part="T3" gate="G$1" x="119.38" y="76.2"/>
+<instance part="C5" gate="G$1" x="-33.02" y="81.28" rot="R90"/>
+<instance part="C6" gate="G$1" x="-33.02" y="66.04" rot="R90"/>
 </instances>
 <busses>
